File: uconsole-expansion-card-template.kicad_sch (KiCad schematic)
At the start: 14 parts, among them U1 UC EXPANSION, U2 Speaker, U3 Speaker

Commit message: Board 1.27mm passes to production!
Parts:
- removed 3V1: Conn_01x02, Connector_PinHeader_1.27mm:PinHeader_1x02_P1.27mm_Vertical, symbol Connector_Generic:Conn_01x02
- removed 5V1: Conn_01x05, Connector_PinHeader_1.27mm:PinHeader_1x05_P1.27mm_Vertical, symbol Connector_Generic:Conn_01x05
- removed CAM1: Conn_01x10, Connector_PinHeader_1.27mm:PinHeader_1x10_P1.27mm_Horizontal, symbol Connector_Generic:Conn_01x10
- removed GPIO1: Conn_01x18, Connector_PinHeader_1.27mm:PinHeader_1x18_P1.27mm_Horizontal, symbol Connector_Generic:Conn_01x18
- removed GROUND1: Conn_01x08, Connector_PinHeader_1.27mm:PinHeader_1x08_P1.27mm_Vertical, symbol Connector_Generic:Conn_01x08
- removed SPK_L1, SPK_R1, USB3, USB4: Conn_01x02, Connector_PinHeader_1.27mm:PinHeader_1x02_P1.27mm_Horizontal, symbol Connector_Generic:Conn_01x02
- added 16_52, 17_51: Conn_01x18, symbol Connector_Generic:Conn_01x18
- added 1_15, 2_16: Conn_01x08, symbol Connector_Generic:Conn_01x08
Connections:
- net +3V3: now also 17_51.1 (Pin_1), 17_51.2 (Pin_2)
- net +5V: now also 2_16.1 (Pin_1), 2_16.2 (Pin_2), 2_16.3 (Pin_3), 2_16.4 (Pin_4), 2_16.5 (Pin_5)
- net CAM1_CN: now also 17_51.11 (Pin_11)
- net CAM1_CP: now also 17_51.10 (Pin_10)
- net CAM1_DN0: now also 17_51.17 (Pin_17)
- net CAM1_DN1: now also 17_51.14 (Pin_14)
- net CAM1_DN2: now also 17_51.8 (Pin_8)
- net CAM1_DN3: now also 17_51.5 (Pin_5)
- net CAM1_DP0: now also 17_51.16 (Pin_16)
- net CAM1_DP1: now also 17_51.13 (Pin_13)
- net CAM1_DP2: now also 17_51.7 (Pin_7)
- net CAM1_DP3: now also 17_51.4 (Pin_4)
- net GND: now also 17_51.12 (Pin_12), 17_51.15 (Pin_15), 17_51.18 (Pin_18), 17_51.3 (Pin_3), 17_51.6 (Pin_6), 17_51.9 (Pin_9), 1_15.3 (Pin_3), 1_15.6 (Pin_6), 2_16.6 (Pin_6)
- net GPIO28: now also 16_52.1 (Pin_1)
- net GPIO29: now also 16_52.2 (Pin_2)
- net GPIO30: now also 16_52.3 (Pin_3)
- net GPIO31: now also 16_52.4 (Pin_4)
- net GPIO32: now also 16_52.5 (Pin_5)
- net GPIO33: now also 16_52.6 (Pin_6)
- net GPIO34: now also 16_52.7 (Pin_7)
- net GPIO35: now also 16_52.8 (Pin_8)
- net GPIO36: now also 16_52.9 (Pin_9)
- net GPIO37: now also 16_52.10 (Pin_10)
- net GPIO38: now also 16_52.11 (Pin_11)
- net GPIO39: now also 16_52.12 (Pin_12)
- net GPIO40: now also 16_52.13 (Pin_13)
- net GPIO41: now also 16_52.14 (Pin_14)
- net GPIO42: now also 16_52.15 (Pin_15)
- net GPIO43: now also 16_52.16 (Pin_16)
- net GPIO44: now also 16_52.17 (Pin_17)
- net GPIO45: now also 16_52.18 (Pin_18)
- net SPEAKER_LN: now also 1_15.2 (Pin_2)
- net SPEAKER_LP: now also 1_15.1 (Pin_1)
- net SPEAKER_RN: now also 2_16.8 (Pin_8)
- net SPEAKER_RP: now also 2_16.7 (Pin_7)
- net USB3_D+: now also 1_15.4 (Pin_4)
- net USB3_D-: now also 1_15.5 (Pin_5)
- net USB4_D+: now also 1_15.7 (Pin_7)
- net USB4_D-: now also 1_15.8 (Pin_8)
Other:
- moved on the sheet: U1
