File: uconsole-expansion-card-template.kicad_pcb_2.54.kicad_pcb (KiCad board)
At the start: 2 copper layers, 35.8 x 77 mm, 231 parts, among them U1 UC EXPANSION, U2 Speaker, U3 Speaker

Commit message: Second Batch
Parts:
- removed the 1 at (86.4, 84.3)
- removed the 100 at (96.6, 122.5)
- removed the 100 at (96.6, 76.5)
- removed the 101 at (99.1, 76.5)
- removed the 101 at (99.1, 122.5)
- removed the 102 at (101.7, 122.5)
- removed the 102 at (101.7, 76.5)
- removed the 103 at (104.2, 76.5)
- removed the 103 at (104.2, 122.5)
- removed the 104 at (106.7, 122.5)
- removed the 104 at (106.7, 76.5)
- removed the 105 at (109.3, 122.5)
- removed the 105 at (109.3, 76.5)
- removed the 106 at (111.8, 76.5)
- removed the 106 at (111.8, 122.5)
- removed the 107 at (83.9, 125.0)
- removed the 107 at (83.9, 79.0)
- removed the 108 at (86.4, 125.0)
- removed the 108 at (86.4, 79.0)
- removed the 109 at (89.0, 125.0)
- removed the 109 at (89.0, 79.0)
- removed the 110 at (91.5, 125.0)
- removed the 110 at (91.5, 79.0)
- removed the 111 at (94.0, 125.0)
- removed the 111 at (94.0, 79.0)
- removed the 112 at (96.6, 79.0)
- removed the 112 at (96.6, 125.0)
- removed the 113 at (99.1, 79.0)
- removed the 113 at (99.1, 125.0)
- removed the 114 at (101.7, 125.0)
- removed the 114 at (101.7, 79.0)
- removed the 115 at (104.2, 125.0)
- removed the 115 at (104.2, 79.0)
- removed the 116 at (106.7, 125.0)
- removed the 116 at (106.7, 79.0)
- removed the 117 at (109.3, 125.0)
- removed the 117 at (109.3, 79.0)
- removed the 118 at (111.8, 125.0)
- removed the 118 at (111.8, 79.0)
- removed the 119 at (83.9, 81.6)
- removed the 119 at (99.1, 117.4)
- removed the 120 at (101.7, 117.4)
- removed the 120 at (86.4, 81.6)
- removed the 121 at (104.2, 117.4)
- removed the 121 at (89.0, 81.6)
- removed the 122 at (106.7, 117.4)
- removed the 122 at (91.5, 81.6)
- removed the 123 at (94.0, 81.6)
- removed the 123 at (109.3, 117.4)
- removed the 124 at (111.8, 117.4)
- removed the 124 at (96.6, 81.6)
- removed the 2 at (89.0, 84.3)
- removed the 3 at (91.5, 84.3)
- removed the 4 at (94.0, 84.3)
- removed the 5 at (83.9, 74.0)
- removed the 5 at (83.9, 119.9)
- removed the 5 at (96.6, 84.3)
- removed the 6 at (83.9, 86.8)
- removed the 7 at (86.4, 86.8)
- removed the 8 at (89.0, 86.8)
- removed the 84 at (86.4, 74.0)
- removed the 84 at (86.4, 119.9)
- removed the 85 at (89.0, 74.0)
- removed the 85 at (89.0, 119.9)
- removed the 86 at (91.5, 119.9)
- removed the 86 at (91.5, 74.0)
- removed the 87 at (94.0, 74.0)
- removed the 87 at (94.0, 119.9)
- removed the 88 at (96.6, 74.0)
- removed the 88 at (96.6, 119.9)
- removed the 89 at (99.1, 74.0)
- removed the 89 at (99.1, 119.9)
- removed the 90 at (101.7, 74.0)
- removed the 90 at (101.7, 119.9)
- removed the 91 at (104.2, 119.9)
- removed the 91 at (104.2, 74.0)
- removed the 92 at (106.7, 74.0)
- removed the 92 at (106.7, 119.9)
- removed the 93 at (109.3, 74.0)
- removed the 93 at (109.3, 119.9)
- removed the 94 at (111.8, 74.0)
- removed the 94 at (111.8, 119.9)
- removed the 95 at (83.9, 122.5)
- removed the 95 at (83.9, 76.5)
- removed the 96 at (86.4, 122.5)
- removed the 96 at (86.4, 76.5)
- removed the 97 at (89.0, 76.5)
- removed the 97 at (89.0, 122.5)
- removed the 98 at (91.5, 76.5)
- removed the 98 at (91.5, 122.5)
- removed the 99 at (94.0, 122.5)
- removed the 99 at (94.0, 76.5)
- removed the ? at (100.4, 85.4)
- removed the ? at (105.2, 85.4)
- removed the ? at (83.9, 84.3)
- removed the ? at (112.4, 114.1)
- removed the ? at (103.6, 85.4)
- removed the ? at (106.0, 85.4)
- removed the ? at (109.2, 114.1)
- removed the ? at (111.6, 85.4)
- removed the ? at (107.6, 114.1)
- removed the ? at (98.8, 85.4)
- removed the ? at (110.8, 114.1)
- removed the ? at (108.4, 85.4)
- removed the ? at (112.4, 85.4)
- removed the ? at (109.2, 85.4)
- removed the ? at (107.6, 85.4)
- removed the ? at (104.4, 85.4)
- removed the ? at (111.6, 114.1)
- removed the ? at (101.2, 85.4)
- removed the ? at (99.6, 85.4)
- removed the ? at (106.8, 85.4)
- removed the ? at (99.6, 102.7)
- removed the ? at (100.4, 102.7)
- removed the ? at (102.8, 85.4)
- removed the ? at (108.4, 102.7)
- removed the ? at (110.0, 102.7)
- removed the ? at (104.4, 102.7)
- removed the ? at (104.5, 114.1)
- removed the ? at (106.0, 102.7)
- removed the ? at (112.4, 102.7)
- removed the ? at (102.9, 114.1)
- removed the ? at (107.6, 102.7)
- removed the ? at (102.1, 114.1)
- removed the ? at (99.7, 114.1)
- removed the ? at (110.8, 85.4)
- removed the ? at (105.2, 102.7)
- removed the ? at (106.8, 102.7)
- removed the ? at (110.8, 102.7)
- removed the ? at (103.6, 102.7)
- removed the ? at (100.5, 114.1)
- removed the ? at (101.2, 102.7)
- removed the ? at (102.8, 102.7)
- removed the ? at (102.0, 102.7)
- removed the ? at (98.9, 114.1)
- removed the ? at (111.6, 102.7)
- removed the ? at (110.0, 114.1)
- removed the ? at (103.7, 114.1)
- removed the ? at (109.2, 102.7)
- removed the ? at (101.3, 114.1)
- removed the ? at (106.8, 114.1)
- removed the ? at (110.0, 85.4)
- removed the ? at (102.0, 85.4)
- removed the ? at (108.4, 114.1)
- removed GPIO45: , 
- added 1: , , F.Cu at (100.4, 104.8)
- added 1: , , F.Cu at (100.4, 85.8)
- added 1: , , F.Cu at (99.4, 103.3)
- added 1: , , F.Cu at (99.4, 84.3)
- added 100: , , F.Cu at (94.0, 104.4)
- added 101: , , F.Cu at (83.8, 107.0)
- added 102: , , F.Cu at (86.3, 107.0)
- added 103: , , F.Cu at (88.9, 107.0)
- added 104: , , F.Cu at (91.4, 107.0)
- added 105: , , F.Cu at (94.0, 107.0)
- added 106: , , F.Cu at (83.8, 109.5)
- added 107: , , F.Cu at (86.3, 109.5)
- added 108: , , F.Cu at (88.9, 109.5)
- added 109: , , F.Cu at (91.4, 109.5)
- added 110: , , F.Cu at (94.0, 109.5)
- added 111: , , F.Cu at (83.8, 112.1)
- added 112: , , F.Cu at (86.3, 112.1)
- added 113: , , F.Cu at (88.9, 112.1)
- added 114: , , F.Cu at (91.4, 112.1)
- added 115: , , F.Cu at (94.0, 112.1)
- added 116: , , F.Cu at (83.8, 114.6)
- added 117: , , F.Cu at (86.3, 114.6)
- added 118: , , F.Cu at (88.9, 114.6)
- added 119: , , F.Cu at (91.4, 114.6)
- added 120: , , F.Cu at (94.0, 114.6)
- added 121: , , F.Cu at (83.8, 117.1)
- added 122: , , F.Cu at (86.3, 117.1)
- added 123: , , F.Cu at (88.9, 117.1)
- added 124: , , F.Cu at (91.4, 117.1)
- added 131: , , F.Cu at (83.8, 122.2)
- added 132: , , F.Cu at (86.3, 122.2)
- added 133: , , F.Cu at (88.9, 122.2)
- added 134: , , F.Cu at (91.4, 122.2)
- added 135: , , F.Cu at (94.0, 122.2)
- added 136: , , F.Cu at (83.8, 124.8)
- added 137: , , F.Cu at (86.3, 124.8)
- added 138: , , F.Cu at (88.9, 124.8)
- added 139: , , F.Cu at (91.4, 124.8)
- added 140: , , F.Cu at (94.0, 124.8)
- added 143: , , F.Cu at (96.5, 89.2)
- added 144: , , F.Cu at (96.5, 91.7)
- added 145: , , F.Cu at (96.5, 94.3)
- added 146: , , F.Cu at (96.5, 107.0)
- added 147: , , F.Cu at (96.5, 109.5)
- added 148: , , F.Cu at (96.5, 112.1)
- added 149: , , F.Cu at (96.5, 114.6)
- added 150: , , F.Cu at (96.5, 117.1)
- added 151: , , F.Cu at (96.5, 119.7)
- added 152: , , F.Cu at (96.5, 122.2)
- added 153: , , F.Cu at (96.5, 124.8)
- added 154: , , F.Cu at (96.5, 96.8)
- added 155: , , F.Cu at (99.0, 117.1)
- added 156: , , F.Cu at (99.0, 119.7)
- added 157: , , F.Cu at (99.0, 122.2)
- added 158: , , F.Cu at (99.0, 124.8)
- added 159: , , F.Cu at (96.5, 99.4)
- added 160: , , F.Cu at (101.6, 117.1)
- added 161: , , F.Cu at (101.6, 119.7)
- added 162: , , F.Cu at (101.6, 122.2)
- added 163: , , F.Cu at (101.6, 124.8)
- added 165: , , F.Cu at (104.1, 117.1)
- added 166: , , F.Cu at (104.1, 119.7)
- added 167: , , F.Cu at (104.1, 122.2)
- added 168: , , F.Cu at (104.1, 124.8)
- added 170: , , F.Cu at (106.7, 117.1)
- added 171: , , F.Cu at (106.7, 119.7)
- added 172: , , F.Cu at (106.7, 122.2)
- added 173: , , F.Cu at (106.7, 124.8)
- added 175: , , F.Cu at (109.2, 117.1)
- added 176: , , F.Cu at (109.2, 119.7)
- added 177: , , F.Cu at (109.2, 122.2)
- added 178: , , F.Cu at (109.2, 124.8)
- added 180: , , F.Cu at (111.8, 117.1)
- added 181: , , F.Cu at (111.8, 119.7)
- added 182: , , F.Cu at (111.8, 122.2)
- added 183: , , F.Cu at (111.8, 124.8)
- added 2: , , F.Cu at (101.2, 103.3)
- added 2: , , F.Cu at (102.2, 85.8)
- added 2: , , F.Cu at (102.2, 104.8)
- added 2: , , F.Cu at (101.2, 84.3)
- added 3: , , F.Cu at (104.0, 104.8)
- added 3: , , F.Cu at (103.0, 84.3)
- added 3: , , F.Cu at (103.0, 103.3)
- added 3: , , F.Cu at (104.0, 85.8)
- added 4: , , F.Cu at (105.8, 104.8)
- added 4: , , F.Cu at (105.8, 85.8)
- added 4: , , F.Cu at (104.8, 103.3)
- added 4: , , F.Cu at (104.8, 84.3)
- added 5: , , F.Cu at (106.6, 84.3)
- added 5: , , F.Cu at (107.6, 85.8)
- added 5: , , F.Cu at (107.6, 104.8)
- added 5: , , F.Cu at (106.6, 103.3)
- added 6: , , F.Cu at (109.4, 104.8)
- added 6: , , F.Cu at (108.4, 84.3)
- added 6: , , F.Cu at (108.4, 103.3)
- added 6: , , F.Cu at (109.4, 85.8)
- added 7: , , F.Cu at (110.2, 103.3)
- added 7: , , F.Cu at (111.2, 85.8)
- added 7: , , F.Cu at (111.2, 104.8)
- added 7: , , F.Cu at (110.2, 84.3)
- added 8: , , F.Cu at (112.0, 103.3)
- added 8: , , F.Cu at (113.0, 104.8)
- added 8: , , F.Cu at (112.0, 84.3)
- added 8: , , F.Cu at (113.0, 85.8)
- added 84: , , F.Cu at (91.4, 96.8)
- added 85: , , F.Cu at (94.0, 96.8)
- added 86: , , F.Cu at (83.8, 99.4)
- added 87: , , F.Cu at (86.3, 99.4)
- added 88: , , F.Cu at (88.9, 99.4)
- added 89: , , F.Cu at (91.4, 99.4)
- added 90: , , F.Cu at (94.0, 99.4)
- added 91: , , F.Cu at (83.8, 101.9)
- added 92: , , F.Cu at (86.3, 101.9)
- added 93: , , F.Cu at (88.9, 101.9)
- added 94: , , F.Cu at (91.4, 101.9)
- added 95: , , F.Cu at (94.0, 101.9)
- added 96: , , F.Cu at (83.8, 104.4)
- added 97: , , F.Cu at (86.3, 104.4)
- added 98: , , F.Cu at (88.9, 104.4)
- added 99: , , F.Cu at (91.4, 104.4)
- added ?: , , F.Cu at (113.3, 114.2)
- added ?: , , F.Cu at (108.5, 112.7)
- added ?: , , F.Cu at (100.9, 112.7)
- added ?: , , F.Cu at (107.6, 114.2)
- added ?: , , F.Cu at (105.5, 114.2)
- added ?: , , F.Cu at (104.7, 112.7)
- added ?: , , F.Cu at (97.6, 103.3)
- added ?: , , F.Cu at (98.6, 85.8)
- added ?: , , F.Cu at (106.6, 112.7)
- added ?: , , F.Cu at (109.5, 114.2)
- added ?: , , F.Cu at (111.4, 114.2)
- added ?: , , F.Cu at (83.8, 74.0)
- added ?: , , F.Cu at (102.8, 112.7)
- added ?: , , F.Cu at (112.3, 112.7)
- added ?: , , F.Cu at (100.0, 114.2)
- added ?: , , F.Cu at (97.6, 84.3)
- added ?: , , F.Cu at (98.6, 104.8)
- added ?: , , F.Cu at (99.0, 112.7)
- added ?: , , F.Cu at (101.9, 114.2)
- added ?: , , F.Cu at (103.7, 114.2)
- added ?: , , F.Cu at (110.4, 112.7)
- moved 127 42.1 mm to (86.3, 119.7)
- moved 130 42.1 mm to (94.0, 119.7)
- moved 126 42.1 mm to (83.8, 119.7)
- moved 128 42.1 mm to (88.9, 119.7)
- moved 129 42.1 mm to (91.4, 119.7)
- moved 54 36.0 mm to (109.2, 81.6)
- moved 55 36.0 mm to (111.8, 81.6)
- moved 125 35.9 mm to (94.0, 117.1)
- moved 42 34.2 mm to (109.2, 79.0)
- moved 43 34.2 mm to (111.8, 79.0)
- moved 30 32.6 mm to (109.2, 76.5)
- moved 31 32.6 mm to (111.8, 76.5)
- moved 18 31.0 mm to (109.2, 74.0)
- moved 19 31.0 mm to (111.8, 74.0)
- moved 60 27.5 mm to (94.0, 84.1)
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Routing:
- net GND: track 129.4 -> 132.5 mm
- net +3V3: track 49.8 -> 52.7 mm
- net /GPIO44: track 30.3 -> 32.4 mm
- net /GPIO30: track 8.27 -> 10.4 mm
- net /GPIO36: track 17.7 -> 19.7 mm
- net /GPIO34: track 14.5 -> 16.5 mm
- net /SPEAKER_RN: track 100.9 -> 98.9 mm
- net /GPIO42: track 27.3 -> 29.2 mm
- net /GPIO32: track 11.5 -> 13.4 mm
- net /GPIO38: track 20.9 -> 22.8 mm
- net /GPIO40: track 24.2 -> 26.0 mm
- net /CAM1_DN3: track 20.7 -> 22.6 mm
- net /SPEAKER_LN: track 47.2 -> 48.9 mm
- net /CAM1_DP2: track 18.6 -> 20.2 mm
- net /USB4_D+: track 15.2 -> 13.7 mm
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