File: uconsole-expansion-card-template_1.27.kicad_pcb (KiCad board)
At the start: 2 copper layers, 35.8 x 77 mm, 627 parts, among them U1 UC EXPANSION, U2 Speaker, U3 Speaker

Commit message: Second Batch
Parts:
- removed the ? at (102.0, 85.4)
- removed the ? at (108.4, 114.1)
- removed the ? at (105.2, 85.4)
- removed the ? at (112.4, 114.1)
- removed the ? at (103.6, 85.4)
- removed the ? at (106.0, 85.4)
- removed the ? at (100.4, 85.4)
- removed the ? at (108.4, 85.4)
- removed the ? at (109.2, 114.1)
- removed the ? at (111.6, 85.4)
- removed the ? at (107.6, 114.1)
- removed the ? at (98.8, 85.4)
- removed the ? at (110.8, 114.1)
- removed the ? at (112.4, 85.4)
- removed the ? at (109.2, 85.4)
- removed the ? at (107.6, 85.4)
- removed the ? at (102.8, 85.4)
- removed the ? at (104.4, 85.4)
- removed the ? at (111.6, 114.1)
- removed the ? at (110.8, 85.4)
- removed the ? at (101.2, 85.4)
- removed the ? at (99.6, 85.4)
- removed the ? at (106.8, 85.4)
- removed the ? at (99.6, 102.7)
- removed the ? at (100.4, 102.7)
- removed the ? at (108.4, 102.7)
- removed the ? at (110.0, 102.7)
- removed the ? at (104.4, 102.7)
- removed the ? at (104.5, 114.1)
- removed the ? at (106.0, 102.7)
- removed the ? at (112.4, 102.7)
- removed the ? at (102.9, 114.1)
- removed the ? at (107.6, 102.7)
- removed the ? at (102.1, 114.1)
- removed the ? at (99.7, 114.1)
- removed the ? at (105.2, 102.7)
- removed the ? at (106.8, 102.7)
- removed the ? at (110.8, 102.7)
- removed the ? at (103.6, 102.7)
- removed the ? at (100.5, 114.1)
- removed the ? at (101.2, 102.7)
- removed the ? at (102.8, 102.7)
- removed the ? at (102.0, 102.7)
- removed the ? at (98.9, 114.1)
- removed the ? at (111.6, 102.7)
- removed the ? at (103.7, 114.1)
- removed the ? at (109.2, 102.7)
- removed the ? at (101.3, 114.1)
- removed the ? at (110.0, 114.1)
- removed the ? at (106.8, 114.1)
- removed the ? at (110.0, 85.4)
- removed GPIO45: , 
- added 1: , , F.Cu at (100.4, 104.8)
- added 1: , , F.Cu at (100.4, 85.8)
- added 1: , , F.Cu at (99.4, 103.3)
- added 1: , , F.Cu at (99.4, 84.3)
- added 10: , , F.Cu at (97.3, 108.0)
- added 11: , , F.Cu at (97.3, 109.3)
- added 12: , , F.Cu at (97.3, 110.7)
- added 13: , , F.Cu at (97.3, 112.1)
- added 14: , , F.Cu at (97.3, 113.4)
- added 15: , , F.Cu at (97.3, 114.8)
- added 2: , , F.Cu at (101.2, 103.3)
- added 2: , , F.Cu at (102.2, 85.8)
- added 2: , , F.Cu at (102.2, 104.8)
- added 2: , , F.Cu at (101.2, 84.3)
- added 3: , , F.Cu at (104.0, 104.8)
- added 3: , , F.Cu at (103.0, 84.3)
- added 3: , , F.Cu at (103.0, 103.3)
- added 3: , , F.Cu at (104.0, 85.8)
- added 4: , , F.Cu at (105.8, 104.8)
- added 4: , , F.Cu at (105.8, 85.8)
- added 4: , , F.Cu at (104.8, 103.3)
- added 4: , , F.Cu at (104.8, 84.3)
- added 5: , , F.Cu at (106.6, 84.3)
- added 5: , , F.Cu at (107.6, 85.8)
- added 5: , , F.Cu at (107.6, 104.8)
- added 5: , , F.Cu at (106.6, 103.3)
- added 6: , , F.Cu at (109.4, 104.8)
- added 6: , , F.Cu at (108.4, 84.3)
- added 6: , , F.Cu at (108.4, 103.3)
- added 6: , , F.Cu at (109.4, 85.8)
- added 7: , , F.Cu at (110.2, 103.3)
- added 7: , , F.Cu at (111.2, 85.8)
- added 7: , , F.Cu at (111.2, 104.8)
- added 7: , , F.Cu at (110.2, 84.3)
- added 8: , , F.Cu at (112.0, 103.3)
- added 8: , , F.Cu at (113.0, 104.8)
- added 8: , , F.Cu at (112.0, 84.3)
- added 8: , , F.Cu at (113.0, 85.8)
- added 9: , , F.Cu at (97.3, 106.6)
- added ?: , , F.Cu at (101.9, 114.2)
- added ?: , , F.Cu at (103.7, 114.2)
- added ?: , , F.Cu at (110.4, 112.7)
- added ?: , , F.Cu at (108.5, 112.7)
- added ?: , , F.Cu at (100.9, 112.7)
- added ?: , , F.Cu at (107.6, 114.2)
- added ?: , , F.Cu at (113.3, 114.2)
- added ?: , , F.Cu at (105.5, 114.2)
- added ?: , , F.Cu at (104.7, 112.7)
- added ?: , , F.Cu at (97.6, 103.3)
- added ?: , , F.Cu at (98.6, 85.8)
- added ?: , , F.Cu at (106.6, 112.7)
- added ?: , , F.Cu at (109.5, 114.2)
- added ?: , , F.Cu at (100.0, 114.2)
- added ?: , , F.Cu at (97.6, 84.3)
- added ?: , , F.Cu at (111.4, 114.2)
- added ?: , , F.Cu at (102.8, 112.7)
- added ?: , , F.Cu at (98.6, 104.8)
- added ?: , , F.Cu at (112.3, 112.7)
- added ?: , , F.Cu at (99.0, 112.7)
Routing:
- net GND: track 129.4 -> 132.5 mm
- net +3V3: track 49.8 -> 52.7 mm
- net /SPEAKER_RN: track 101.5 -> 98.9 mm
- net /GPIO44: track 30.3 -> 32.4 mm
- net /GPIO30: track 8.27 -> 10.4 mm
- net /GPIO36: track 17.7 -> 19.7 mm
- net /GPIO34: track 14.5 -> 16.5 mm
- net /GPIO42: track 27.3 -> 29.2 mm
- net /GPIO32: track 11.5 -> 13.4 mm
- net /GPIO38: track 20.9 -> 22.8 mm
- net /GPIO40: track 24.2 -> 26.0 mm
- net /CAM1_DN3: track 20.7 -> 22.6 mm
- net /CAM1_DP2: track 18.6 -> 20.2 mm
- net /USB4_D+: track 15.3 -> 13.7 mm
- net /GPIO28: track 7.10 -> 5.54 mm
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